File: LogicBoard/rgb_display.kicad_sch (KiCad schematic)
At the start: 1 part, among them J1 Conn_01x50

Commit message: Created display psu layout
Connections:
- net Bus_Disp_pwr.LED_K is gone; now on net GND: J1.3 (Pin_3), J1.4 (Pin_4)
Changed lines of the file:
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@@
 	(paper "A4")
+	(junction
+		(at 39.37 54.61)
+		(diameter 0)
+		(color 0 0 0 0)
+	)
+	(junction
+		(at 39.37 52.07)
+		(diameter 0)
+		(color 0 0 0 0)
+	)
 	(junction
 		(at 39.37 44.45)
@@
 	(wire
 		(pts
-			(xy 41.91 54.61) (xy 36.83 54.61)
+			(xy 41.91 54.61) (xy 39.37 54.61)
 		)
 		(stroke
@@
 	(wire
 		(pts
+			(xy 39.37 54.61) (xy 39.37 52.07)
+		)
+		(stroke
+			(width 0)
+			(type default)
+		)
+	)
+	(wire
+		(pts
 			(xy 39.37 52.07) (xy 39.37 49.53)
 		)
@@
 		(pts
 			(xy 36.83 147.955) (xy 80.645 147.955)
+		)
+		(stroke
+			(width 0)
+			(type default)
+		)
+	)
+	(wire
+		(pts
+			(xy 39.37 54.61) (xy 36.83 54.61)
 		)
 		(stroke
@@
 	)
 	(label "Bus_Disp_control.DITHB"
-		(at 47.625 161.29 0)
-		(effects
-			(font
-				(size 1.27 1.27)
-			)
-			(justify left bottom)
+		(at 47.625 161.29 180)
+		(effects
+			(font
+				(size 1.27 1.27)
+			)
+			(justify right bottom)
 		)
 	)
@@
 	)
 	(label "Bus_Disp_pwr.VCOM"
-		(at 50.8 158.115 0)
-		(effects
-			(font
-				(size 1.27 1.27)
-			)
-			(justify left bottom)
-		)
-	)
+		(at 50.8 158.115 180)
+		(effects
+			(font
+				(size 1.27 1.27)
+			)
+			(justify right bottom)
+		)
+	)
