File: LogicBoard/PowerSection.kicad_sch (KiCad schematic)
At the start: 45 parts, among them U2 TPS65150PWPR, U4 TPS54331DR

Commit message: experimenting with bga
Parts:
- D1, D2, D3, D4, D5, D6: value 1N5818 -> MBRS130LT3G; footprint Diode_SMD:D_SOD-123F -> Diode_SMD:D_SMB; jlcpcbpart C437955 -> C51771
Changed lines of the file:
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@@
 			)
 		)
-		(property "Value" "1N5818"
+		(property "Value" "MBRS130LT3G"
 			(at 311.4675 185.42 0)
 			(show_name no)
@@
 			)
 		)
-		(property "Footprint" "Diode_SMD:D_SOD-123F"
+		(property "Footprint" "Diode_SMD:D_SMB"
 			(at 311.15 193.675 0)
 			(hide yes)
@@
 			)
 		)
-		(property "Datasheet" "http://www.vishay.com/docs/88525/1n5817.pdf"
+		(property "Datasheet" ""
 			(at 311.15 189.23 0)
 			(hide yes)
@@
 			)
 		)
-		(property "jlcpcbpart" "C437955"
+		(property "jlcpcbpart" "C51771"
 			(at 311.15 189.23 0)
 			(hide yes)
@@
 			)
 		)
-		(property "Value" "1N5818"
+		(property "Value" "MBRS130LT3G"
 			(at 308.9275 193.04 0)
 			(show_name no)
@@
 			)
 		)
-		(property "Footprint" "Diode_SMD:D_SOD-123F"
+		(property "Footprint" "Diode_SMD:D_SMB"
 			(at 308.61 191.77 0)
 			(hide yes)
@@
 			)
 		)
-		(property "Datasheet" "http://www.vishay.com/docs/88525/1n5817.pdf"
+		(property "Datasheet" ""
 			(at 308.61 196.215 0)
 			(hide yes)
@@
 			)
 		)
-		(property "jlcpcbpart" "C437955"
+		(property "jlcpcbpart" "C51771"
 			(at 308.61 196.215 0)
 			(hide yes)
@@
 			)
 		)
-		(property "Value" "1N5818"
+		(property "Value" "MBRS130LT3G"
 			(at 209.8675 177.165 0)
 			(show_name no)
@@
 			)
 		)
-		(property "Footprint" "Diode_SMD:D_SOD-123F"
+		(property "Footprint" "Diode_SMD:D_SMB"
 			(at 209.55 176.53 0)
 			(hide yes)
@@
 			)
 		)
-		(property "Datasheet" "http://www.vishay.com/docs/88525/1n5817.pdf"
+		(property "Datasheet" ""
 			(at 209.55 180.975 0)
 			(hide yes)
@@
 			)
 		)
-		(property "jlcpcbpart" "C437955"
+		(property "jlcpcbpart" "C51771"
 			(at 209.55 180.975 0)
 			(hide yes)
@@
 			)
 		)
-		(property "Value" "1N5818"
+		(property "Value" "MBRS130LT3G"
 			(at 278.4475 154.94 0)
 			(show_name no)
@@
 			)
 		)
-		(property "Footprint" "Diode_SMD:D_SOD-123F"
+		(property "Footprint" "Diode_SMD:D_SMB"
 			(at 278.13 154.305 0)
 			(hide yes)
@@
 			)
 		)
-		(property "Datasheet" "http://www.vishay.com/docs/88525/1n5817.pdf"
+		(property "Datasheet" ""
 			(at 278.13 158.75 0)
 			(hide yes)
@@
 			)
 		)
-		(property "jlcpcbpart" "C437955"
+		(property "jlcpcbpart" "C51771"
 			(at 278.13 158.75 0)
 			(hide yes)
@@
 			)
 		)
-		(property "Value" "1N5818"
+		(property "Value" "MBRS130LT3G"
 			(at 147.32 57.15 90)
 			(show_name no)
@@
 			)
 		)
-		(property "Footprint" "Diode_SMD:D_SOD-123F"
+		(property "Footprint" "Diode_SMD:D_SMB"
 			(at 152.4 55.88 0)
 			(hide yes)
@@
 			)
 		)
-		(property "Datasheet" "http://www.vishay.com/docs/88525/1n5817.pdf"
+		(property "Datasheet" ""
 			(at 156.845 55.88 0)
 			(hide yes)
@@
 			)
 		)
-		(property "jlcpcbpart" "C437955"
+		(property "jlcpcbpart" "C51771"
 			(at 156.845 55.88 0)
 			(hide yes)
@@
 			)
 		)
-		(property "Value" "1N5818"
+		(property "Value" "MBRS130LT3G"
 			(at 219.71 188.2774 90)
 			(show_name no)
@@
 			)
 		)
-		(property "Footprint" "Diode_SMD:D_SOD-123F"
+		(property "Footprint" "Diode_SMD:D_SMB"
 			(at 221.615 186.69 0)
 			(hide yes)
@@
 			)
 		)
-		(property "Datasheet" "http://www.vishay.com/docs/88525/1n5817.pdf"
+		(property "Datasheet" ""
 			(at 217.17 186.69 0)
 			(hide yes)
@@
 			)
 		)
-		(property "jlcpcbpart" "C437955"
+		(property "jlcpcbpart" "C51771"
 			(at 217.17 186.69 90)
 			(hide yes)
