File: LogicBoard/mcu.kicad_sch (KiCad schematic)
At the start: 1 part, among them U1 STM32H757XIHx

Commit message: added jlcpcb nums to some parts
Changed lines of the file:
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@@
+		)
+	)
+	(hierarchical_label "FLK_CLK"
+		(shape output)
+		(at 65.405 143.51 180)
+		(effects
+			(font
+				(size 1.27 1.27)
+			)
+			(justify right)
 		)
 	)

Commit message: experimenting with bga
Parts:
- added C22, C24: 12p, Capacitor_SMD:C_0402_1005Metric, symbol Device:C_Small
- added Y1: X322525MOB4SI 25MHZ, Crystal:Crystal_SMD_3225-4Pin_3.2x2.5mm, symbol Device:Crystal_GND24
Connections:
- net SDRAM.D25: now reaches U1.A15 (PI1)
- net SDRAM.D24: now reaches U1.A16 (PI0)
- net SDRAM.D28: now reaches U1.A2 (PI6)
- net SDRAM.NBL3: now reaches U1.A3 (PI5)
- net SDRAM.NBL2: now reaches U1.A4 (PI4)
- net SDRAM.D26: now reaches U1.B15 (PI2)
- net SDRAM.D23: now reaches U1.B16 (PH15)
- net SDRAM.D22: now reaches U1.B17 (PH14)
- net SDRAM.D29: now reaches U1.B3 (PI7)
- net SDRAM.NBL1: now reaches U1.B4 (PE1)
- net SDRAM.D27: now reaches U1.C14 (PI3)
- net SDRAM.NBL0: now reaches U1.C4 (PE0)
- net SDRAM.D2: now reaches U1.D13 (PD0)
- net SDRAM.D21: now reaches U1.D16 (PH13)
- net SDRAM.SDNCAS: now reaches U1.D6 (PG15)
- net SDRAM.D3: now reaches U1.E12 (PD1)
- net SDRAM.D30: now reaches U1.E2 (PI9)
- net SDRAM.SDCLK: now reaches U1.F15 (PG8)
- net SDRAM.D31: now reaches U1.F3 (PI10)
- net SDRAM.A2: now reaches U1.G1 (PF2)
- net SDRAM.BA1: now reaches U1.G14 (PG5)
- net SDRAM.A1: now reaches U1.G3 (PF1)
- net SDRAM.A0: now reaches U1.G4 (PF0)
- net SDRAM.BA0: now reaches U1.H14 (PG4)
- net SDRAM.A3: now reaches U1.H4 (PF3)
- net OSC_OUT: now reaches U1.J1 (PH1)
- net OSC_OUT: now also C24.1, Y1.1
- net OSC_IN: now reaches U1.J2 (PH0)
- net OSC_IN: now also C22.1, Y1.3
- net SDRAM.A5: now reaches U1.J4 (PF5)
- net SDRAM.A4: now reaches U1.J5 (PF4)
- net SDRAM.SDNWE: now reaches U1.L2 (PC0)
- net SDRAM.SDNE0: now reaches U1.M3 (PC2)
- net SDRAM.SDCKE0: now reaches U1.M4 (PC3)
- net SDRAM.D7: now reaches U1.N9 (PE10)
- net SDRAM.D8: now reaches U1.P10 (PE11)
- net SDRAM.D18: now reaches U1.P13 (PH10)
- net SDRAM.D19: now reaches U1.P14 (PH11)
- net SDRAM.D1: now reaches U1.P15 (PD15)
- net SDRAM.D0: now reaches U1.P16 (PD14)
- net SDRAM.A7: now reaches U1.P7 (PF13)
- net SDRAM.A8: now reaches U1.P8 (PF14)
- net SDRAM.D6: now reaches U1.P9 (PE9)
- net SDRAM.D9: now reaches U1.R10 (PE12)
- net SDRAM.D12: now reaches U1.R11 (PE15)
- net SDRAM.D17: now reaches U1.R13 (PH9)
- net SDRAM.D20: now reaches U1.R14 (PH12)
- net SDRAM.A6: now reaches U1.R7 (PF12)
- net SDRAM.A9: now reaches U1.R9 (PF15)
- net SDRAM.D10: now reaches U1.T10 (PE13)
- net SDRAM.D16: now reaches U1.T13 (PH8)
- net SDRAM.D15: now reaches U1.T16 (PD10)
- net SDRAM.D14: now reaches U1.T17 (PD9)
- net SDRAM.SDNRAS: now reaches U1.T7 (PF11)
- net SDRAM.A10: now reaches U1.T8 (PG0)
- net SDRAM.D5: now reaches U1.T9 (PE8)
- net SDRAM.D11: now reaches U1.U10 (PE14)
- net SDRAM.D13: now reaches U1.U16 (PD8)
- net SDRAM.A11: now reaches U1.U8 (PG1)
- net SDRAM.D4: now reaches U1.U9 (PE7)
- new net GND: C22.2, C24.2, Y1.2 (G), Y1.4 (G)
Other:
- note added: "CLK"
- moved on the sheet: U1
