File: AudioBoard/AudioBoard/codec.kicad_sch (KiCad schematic)
At the start: 0 parts

Commit message: Created input sections
Parts:
- added C228, C68: 1nF, Capacitor_SMD:C_0603_1608Metric, symbol Device:C_Small
- added C57, C79: 100nF, Capacitor_SMD:C_0603_1608Metric, symbol Device:C_Small
- added C58: 100uF tantal, Capacitor_Tantalum_SMD:CP_EIA-3528-21_Kemet-B, symbol Device:C_Polarized_Small_US
- added C67: 33nF, Capacitor_SMD:C_0805_2012Metric_Pad1.18x1.45mm_HandSolder, symbol Device:C_Small
- added C80: 10uF tantal, Capacitor_Tantalum_SMD:CP_EIA-3216-18_Kemet-A, symbol Device:C_Polarized_Small_US
- added R45: 3k, Resistor_SMD:R_0603_1608Metric, symbol Device:R
- added U1: (no value), Package_QFP:LQFP-64_10x10mm_P0.5mm, symbol ad1939_1:AD1939
Connections:
- new net: C67.1, R45.1
- new net +3.3V: U1.14 (PD/RST)
- new net AD1939_CM: C57.2, C58.1, U1.52 (CM)
- new net AD1939_FILTR: C79.2, C80.1, U1.47 (FILTR)
- new net AD1939_LF: C228.2, C67.2, C68.2, U1.61 (LF)
- new net AD1939_MCLKI: U1.2 (MCLKI/XI)
- new net AD1939_MCLKO: U1.3 (MCLKO/XO)
- new net AVDD: C228.1, C68.1, R45.2, U1.45 (AVDD), U1.5 (AVDD), U1.51 (AVDD), U1.62 (AVDD)
- new net DVDD: U1.17 (DVDD), U1.32 (DVDD)
- new net GND: C57.1, C58.2, C79.1, C80.2, U1.1 (AGND), U1.16 (DGND), U1.23 (VSUPPLY), U1.24 (VSENSE), U1.25 (VDRIVE), U1.33 (DGND), U1.4 (AGND), U1.44 (AGND), U1.46 (AGND), U1.48 (AGND)
- new net I2S.CLK: U1.21 (DBCLK), U1.28 (ABCLK)
- new net I2S.SDI: U1.27 (ASDATA1)
- new net I2S.SDO: U1.20 (DSDATA1)
- new net I2S.WS: U1.22 (DLRCLK), U1.29 (ALRCLK)
- new net IN1_N: U1.54 (ADC1LN)
- new net IN1_P: U1.53 (ADC1LP)
- new net IN2_N: U1.56 (ADC1RN)
- new net IN2_P: U1.55 (ADC1RP)
- new net IN3_N: U1.58 (ADC2LN)
- new net IN3_P: U1.57 (ADC2LP)
- new net IN4_N: U1.60 (ADC2RN)
- new net IN4_P: U1.59 (ADC2RP)
- new net OUT1_N: U1.39 (OR1N)
- new net OUT1_P: U1.38 (OR1P)
- new net OUT2_N: U1.37 (OL1N)
- new net OUT2_P: U1.36 (OL1P)
- new net OUT3_N: U1.43 (OR2N)
- new net OUT3_P: U1.42 (OR2P)
- new net OUT4_N: U1.41 (OL2N)
- new net OUT4_P: U1.40 (OL2P)
- new net OUT5_N: U1.9 (OR3N)
- new net OUT5_P: U1.8 (OR3P)
- new net OUT6_N: U1.7 (OL3N)
- new net OUT6_P: U1.6 (OL3P)
- new net OUT7_N: U1.13 (OR4N)
- new net OUT7_P: U1.12 (OR4P)
- new net OUT8_N: U1.11 (OL4N)
- new net OUT8_P: U1.10 (OL4P)
- new net SPI.CLK: U1.34 (CCLK)
- new net SPI.CS: U1.35 (CLATCH)
- new net SPI.MISO: U1.31 (COUT)
- new net SPI.MOSI: U1.30 (CIN)
- no-connect marks 0 -> 4
Other:
- note added: "CM pin filter (can be used for BIAS)"
- note added: "FILTR filtering"
- note added: "MCLK is powered from external quarc osc"
- note added: "PLL Filters"
