File: AudioBoard/AudioBoard/Audio_IO_conn.kicad_sch (KiCad schematic)
At the start: 0 parts

Commit message: added jack IO, headphone amp cirucit
Parts:
- added J1: IN, Connector_Audio:Jack_XLR-6.35mm_Neutrik_NCJ6FA-H_Horizontal, symbol Connector_Audio:NCJ6FA-H
- added J2: XLR_L, Connector_Audio:Jack_XLR_Neutrik_NC3MAH_Horizontal, symbol Connector_Audio:XLR3_Ground
- added J3: FX_RETURN, haoyu:HAOYU_PJ-625, symbol Connector_Audio:AudioJack3_Dual_Ground_Switch
- added J4: FX_SEND, haoyu:HAOYU_PJ-625, symbol Connector_Audio:AudioJack3_Dual_Ground_Switch
- added J5: INS_OUT, haoyu:HAOYU_PJ-625, symbol Connector_Audio:AudioJack3_Dual_Ground_Switch
- added J6: XLR_R, Connector_Audio:Jack_XLR_Neutrik_NC3MAH_Horizontal, symbol Connector_Audio:XLR3_Ground
Connections:
- new net GND: J1.1, J1.G, J1.S, J2.1, J2.G, J3.G, J3.S1, J3.S2, J4.G, J4.S1, J4.S2, J5.G, J5.S1, J5.S2, J6.1, J6.G
- new net OUT_L: J5.T1
- new net OUT_R: J5.T2
- new net RET_1: J3.T1
- new net RET_2: J3.T2
- new net SEND_1: J4.T1
- new net SEND_2: J4.T2
- new net XLR_L_N: J2.3
- new net XLR_L_P: J2.2
- new net XLR_R_N: J6.3
- new net XLR_R_P: J6.2
- new net ins_in: J1.T
- new net xlr_in_n: J1.3
- new net xlr_in_p: J1.2
Other:
- note added: "Combo INPUT XLR/JACK"
- note added: "FX LOOP"
- note added: "INSTRUMENT OUT L(MONO)/R"
- note added: "RETURN"
- note added: "SEND"
- note added: "XLR_OUT"

Commit message: added pwr sw and headphone out
Parts:
- added J8: NMJ6HFD2, Connector_Audio:Jack_6.35mm_Neutrik_NMJ6HFD2_Horizontal, symbol Connector_Audio:NMJ6HFD2
Connections:
- net GND: now also J8.S
- new net HEADPHONE_L: J8.R
- new net HEADPHONE_R: J8.T
Other:
- note added: "HEADPHONE"
Changed lines of the file:
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@@
+	)
+	(rectangle
+		(start 17.145 147.955)
+		(end 97.155 183.515)
+		(stroke
+			(width 0)
+			(type default)
+		)
+		(fill
+			(type none)
+		)
 	)
 	(rectangle
@@
 		(fill
 			(type none)
+		)
+	)
+	(text "HEADPHONE"
+		(exclude_from_sim no)
+		(at 22.86 146.685 0)
+		(effects
+			(font
+				(size 1.27 1.27)
+			)
 		)
 	)
@@
 	(wire
 		(pts
+			(xy 35.56 160.655) (xy 37.465 160.655)
+		)
+		(stroke
+			(width 0)
+			(type default)
+		)
+	)
+	(wire
+		(pts
 			(xy 176.53 81.915) (xy 173.355 81.915)
 		)
@@
 	(wire
 		(pts
+			(xy 35.56 165.735) (xy 37.465 165.735)
+		)
+		(stroke
+			(width 0)
+			(type default)
+		)
+	)
+	(wire
+		(pts
 			(xy 20.955 42.545) (xy 33.655 42.545)
 		)
@@
 	(wire
 		(pts
+			(xy 35.56 155.575) (xy 55.88 155.575)
+		)
+		(stroke
+			(width 0)
+			(type default)
+		)
+	)
+	(wire
+		(pts
 			(xy 48.26 43.815) (xy 36.195 43.815)
 		)
@@
 			(width 0)
 			(type default)
+		)
+	)
+	(hierarchical_label "HEADPHONE_L"
+		(shape input)
+		(at 37.465 160.655 0)
+		(effects
+			(font
+				(size 1.27 1.27)
+			)
+			(justify left)
 		)
 	)
@@
 		(shape input)
 		(at 139.065 43.815 0)
+		(effects
+			(font
+				(size 1.27 1.27)
+			)
+			(justify left)
+		)
+	)
+	(hierarchical_label "HEADPHONE_R"
+		(shape input)
+		(at 37.465 165.735 0)
 		(effects
 			(font
@@
 	(symbol
 		(lib_id "power:GND")
+		(at 55.88 155.575 0)
+		(unit 1)
+		(body_style 1)
+		(exclude_from_sim no)
+		(in_bom yes)
+		(on_board yes)
+		(in_pos_files yes)
+		(dnp no)
+		(fields_autoplaced yes)
+		(property "Reference" "#PWR075"
+			(at 55.88 161.925 0)
+			(hide yes)
+			(show_name no)
+			(do_not_autoplace no)
+			(effects
+				(font
+					(size 1.27 1.27)
+				)
+			)
+		)
+		(property "Value" "GND"
+			(at 55.88 160.655 0)
+			(show_name no)
+			(do_not_autoplace no)
+			(effects
+				(font
+					(size 1.27 1.27)
+				)
+			)
+		)
+		(property "Footprint" ""
+			(at 55.88 155.575 0)
+			(hide yes)
+			(show_name no)
+			(do_not_autoplace no)
+			(effects
+				(font
+					(size 1.27 1.27)
+				)
+			)
+		)
+		(property "Datasheet" ""
+			(at 55.88 155.575 0)
+			(hide yes)
+			(show_name no)
+			(do_not_autoplace no)
+			(effects
+				(font
+					(size 1.27 1.27)
+				)
+			)
+		)
+		(property "Description" "Power symbol creates a global label with name \"GND\" , ground"
+			(at 55.88 155.575 0)
+			(hide yes)
+			(show_name no)
+			(do_not_autoplace no)
+			(effects
+				(font
+					(size 1.27 1.27)
+				)
+			)
+		)
+		(pin "1"
+		)
+		(instances
+			(project "AudioBoard"
+				(path "/dd5d876d-fff7-4cb4-baee-a023036d12ae/6c99cd00-a4a2-4f1f-8c45-97dcde60f012"
+					(reference "#PWR075")
+					(unit 1)
+				)
+			)
+		)
+	)
+	(symbol
+		(lib_id "power:GND")
 		(at 21.59 118.11 0)
 		(unit 1)
@@
 					(unit 1)
 				)
+			)
+		)
+	)
+	(symbol
+		(lib_id "Connector_Audio:NMJ6HFD2")
+		(at 30.48 160.655 0)
+		(unit 1)
+		(body_style 1)
+		(exclude_from_sim no)
+		(in_bom yes)
+		(on_board yes)
+		(in_pos_files yes)
+		(dnp no)
+		(fields_autoplaced yes)
+		(property "Reference" "J8"
+			(at 28.575 149.86 0)
+			(show_name no)
+			(do_not_autoplace no)
+			(effects
+				(font
+					(size 1.27 1.27)
+				)
+			)
+		)
+		(property "Value" "NMJ6HFD2"
+			(at 28.575 152.4 0)
+			(show_name no)
+			(do_not_autoplace no)
+			(effects
+				(font
+					(size 1.27 1.27)
+				)
+			)
+		)
+		(property "Footprint" "Connector_Audio:Jack_6.35mm_Neutrik_NMJ6HFD2_Horizontal"
+			(at 30.48 160.655 0)
+			(hide yes)
+			(show_name no)
+			(do_not_autoplace no)
+			(effects
+				(font
+					(size 1.27 1.27)
+				)
+			)
+		)
+		(property "Datasheet" "https://www.neutrik.com/en/product/nmj6hfd2"
+			(at 30.48 160.655 0)
+			(hide yes)
+			(show_name no)
+			(do_not_autoplace no)
+			(effects
+				(font
+					(size 1.27 1.27)
+				)
+			)
+		)
+		(property "Description" "M Series, 6.35mm (1/4in) stereo jack, switched, with full threaded nose and straight PCB pins"
+			(at 30.48 160.655 0)
+			(hide yes)
+			(show_name no)
+			(do_not_autoplace no)
+			(effects
+				(font
+					(size 1.27 1.27)
+				)
+			)
+		)
+		(pin "SN"
+		)
+		(pin "S"
+		)
+		(pin "R"
+		)
+		(pin "TN"
+		)
+		(pin "RN"
+		)
+		(pin "T"
+		)
+		(instances
+			(project "AudioBoard"
+				(path "/dd5d876d-fff7-4cb4-baee-a023036d12ae/6c99cd00-a4a2-4f1f-8c45-97dcde60f012"
+					(reference "J8")
+					(unit 1)
+				)

Commit message: added connectors to pcb
Parts:
- added J9: NMJ6HFD2, Connector_Audio:Jack_6.35mm_Neutrik_NMJ6HFD2_Horizontal, symbol Connector_Audio:NMJ6HFD2
Connections:
- net GND: now also J9.S
- new net EXP_PWR: J9.T
- new net EXP_SIG: J9.R
Other:
- note added: "EXP_PEDAL_INPUT"
Changed lines of the file:
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@@
 	(paper "A3")
+	(rectangle
+		(start 17.145 182.245)
+		(end 64.77 207.01)
+		(stroke
+			(width 0)
+			(type default)
+		)
+		(fill
+			(type none)
+		)
+	)
 	(rectangle
 		(start 15.875 19.685)
@@
 	(rectangle
 		(start 17.145 147.955)
-		(end 97.155 183.515)
+		(end 64.77 172.72)
 		(stroke
 			(width 0)
@@
 		(exclude_from_sim no)
 		(at 111.125 62.23 0)
+		(effects
+			(font
+				(size 1.27 1.27)
+			)
+		)
+	)
+	(text "EXP_PEDAL_INPUT"
+		(exclude_from_sim no)
+		(at 25.4 180.975 0)
 		(effects
 			(font
@@
 	(wire
 		(pts
+			(xy 35.56 200.025) (xy 37.465 200.025)
+		)
+		(stroke
+			(width 0)
+			(type default)
+		)
+	)
+	(wire
+		(pts
 			(xy 175.895 43.815) (xy 172.72 43.815)
 		)
@@
 	(wire
 		(pts
+			(xy 54.61 189.865) (xy 35.56 189.865)
+		)
+		(stroke
+			(width 0)
+			(type default)
+		)
+	)
+	(wire
+		(pts
 			(xy 46.355 34.29) (xy 43.815 34.29)
 		)
@@
 		(pts
 			(xy 81.28 71.12) (xy 86.36 71.12)
+		)
+		(stroke
+			(width 0)
+			(type default)
+		)
+	)
+	(wire
+		(pts
+			(xy 35.56 194.945) (xy 37.465 194.945)
 		)
 		(stroke
@@
 		)
 	)
+	(hierarchical_label "EXP_PWR"
+		(shape input)
+		(at 37.465 200.025 0)
+		(effects
+			(font
+				(size 1.27 1.27)
+			)
+			(justify left)
+		)
+	)
 	(hierarchical_label "xlr_in_n"
 		(shape output)
@@
 		(shape output)
 		(at 79.375 37.465 0)
+		(effects
+			(font
+				(size 1.27 1.27)
+			)
+			(justify left)
+		)
+	)
+	(hierarchical_label "EXP_SIG"
+		(shape output)
+		(at 37.465 194.945 0)
 		(effects
 			(font
@@
 	(symbol
 		(lib_id "power:GND")
+		(at 54.61 189.865 0)
+		(unit 1)
+		(body_style 1)
+		(exclude_from_sim no)
+		(in_bom yes)
+		(on_board yes)
+		(in_pos_files yes)
+		(dnp no)
+		(fields_autoplaced yes)
+		(property "Reference" "#PWR076"
+			(at 54.61 196.215 0)
+			(hide yes)
+			(show_name no)
+			(do_not_autoplace no)
+			(effects
+				(font
+					(size 1.27 1.27)
+				)
+			)
+		)
+		(property "Value" "GND"
+			(at 54.61 194.945 0)
+			(show_name no)
+			(do_not_autoplace no)
+			(effects
+				(font
+					(size 1.27 1.27)
+				)
+			)
+		)
+		(property "Footprint" ""
+			(at 54.61 189.865 0)
+			(hide yes)
+			(show_name no)
+			(do_not_autoplace no)
+			(effects
+				(font
+					(size 1.27 1.27)
+				)
+			)
+		)
+		(property "Datasheet" ""
+			(at 54.61 189.865 0)
+			(hide yes)
+			(show_name no)
+			(do_not_autoplace no)
+			(effects
+				(font
+					(size 1.27 1.27)
+				)
+			)
+		)
+		(property "Description" "Power symbol creates a global label with name \"GND\" , ground"
+			(at 54.61 189.865 0)
+			(hide yes)
+			(show_name no)
+			(do_not_autoplace no)
+			(effects
+				(font
+					(size 1.27 1.27)
+				)
+			)
+		)
+		(pin "1"
+		)
+		(instances
+			(project "AudioBoard"
+				(path "/dd5d876d-fff7-4cb4-baee-a023036d12ae/6c99cd00-a4a2-4f1f-8c45-97dcde60f012"
+					(reference "#PWR076")
+					(unit 1)
+				)
+			)
+		)
+	)
+	(symbol
+		(lib_id "power:GND")
 		(at 49.53 71.12 0)
 		(unit 1)
@@
 					(unit 1)
 				)
+			)
+		)
+	)
+	(symbol
+		(lib_id "Connector_Audio:NMJ6HFD2")
+		(at 30.48 194.945 0)
+		(unit 1)
+		(body_style 1)
+		(exclude_from_sim no)
+		(in_bom yes)
+		(on_board yes)
+		(in_pos_files yes)
+		(dnp no)
+		(fields_autoplaced yes)
+		(property "Reference" "J9"
+			(at 28.575 184.15 0)
+			(show_name no)
+			(do_not_autoplace no)
+			(effects
+				(font
+					(size 1.27 1.27)
+				)
+			)
+		)
+		(property "Value" "NMJ6HFD2"
+			(at 28.575 186.69 0)
+			(show_name no)
+			(do_not_autoplace no)
+			(effects
+				(font
+					(size 1.27 1.27)
+				)
+			)
+		)
+		(property "Footprint" "Connector_Audio:Jack_6.35mm_Neutrik_NMJ6HFD2_Horizontal"
+			(at 30.48 194.945 0)
+			(hide yes)
+			(show_name no)
+			(do_not_autoplace no)
+			(effects
+				(font
+					(size 1.27 1.27)
+				)
+			)
+		)
+		(property "Datasheet" "https://www.neutrik.com/en/product/nmj6hfd2"
+			(at 30.48 194.945 0)
+			(hide yes)
+			(show_name no)
+			(do_not_autoplace no)
+			(effects
+				(font
+					(size 1.27 1.27)
+				)
+			)
+		)
+		(property "Description" "M Series, 6.35mm (1/4in) stereo jack, switched, with full threaded nose and straight PCB pins"
+			(at 30.48 194.945 0)
+			(hide yes)
+			(show_name no)
+			(do_not_autoplace no)
+			(effects
+				(font
+					(size 1.27 1.27)
+				)
+			)
+		)
+		(pin "SN"
+		)
+		(pin "S"
+		)
+		(pin "R"
+		)
+		(pin "TN"
+		)
+		(pin "RN"
+		)
+		(pin "T"
+		)
+		(instances
+			(project "AudioBoard"
+				(path "/dd5d876d-fff7-4cb4-baee-a023036d12ae/6c99cd00-a4a2-4f1f-8c45-97dcde60f012"
+					(reference "J9")
+					(unit 1)
+				)

Commit message: added lcscpart to components and assigned footprints
Parts:
- J1: JLCPCB (none) -> C368458; LCSC Part (none) -> C368458
- J2, J6: JLCPCB (none) -> C23689430; LCSC Part (none) -> C23689430
- J3, J4, J5: JLCPCB (none) -> C309286; LCSC Part (none) -> C309286
- J8, J9: JLCPCB (none) -> C309279; LCSC Part (none) -> C309279
