File: AudioBoard/AudioBoard/Audio_IO_conn.kicad_sch (KiCad schematic)
At the start: 8 parts, among them J1 IN, J2 XLR_L, J3 FX_RETURN, J4 FX_SEND, J5 INS_OUT, J6 XLR_R, J8 NMJ6HFD2, J9 NMJ6HFD2

Commit message: added first time routing to see crosssections
Changed lines of the file:
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@@
 	)
 	(hierarchical_label "XLR_R_N"
-		(shape output)
+		(shape input)
 		(at 84.455 126.365 0)
 		(effects
@@
 	)
 	(hierarchical_label "XLR_L_N"
-		(shape output)
+		(shape input)
 		(at 45.72 125.73 0)
 		(effects
@@
 	)
 	(hierarchical_label "XLR_L_P"
-		(shape output)
+		(shape input)
 		(at 45.72 123.825 0)
 		(effects
@@
 	)
 	(hierarchical_label "SEND_2"
-		(shape output)
+		(shape input)
 		(at 176.53 81.915 0)
 		(effects
@@
 	)
 	(hierarchical_label "RET_1"
-		(shape input)
+		(shape output)
 		(at 139.065 43.815 0)
 		(effects
@@
 	)
 	(hierarchical_label "OUT_R"
-		(shape output)
+		(shape input)
 		(at 84.455 81.28 0)
 		(effects
@@
 	)
 	(hierarchical_label "XLR_R_P"
-		(shape output)
+		(shape input)
 		(at 84.455 124.46 0)
 		(effects
@@
 	)
 	(hierarchical_label "RET_2"
-		(shape input)
+		(shape output)
 		(at 175.895 43.815 0)
 		(effects
@@
 	)
 	(hierarchical_label "SEND_1"
-		(shape output)
+		(shape input)
 		(at 139.7 81.915 0)
 		(effects
@@
 	)
 	(hierarchical_label "OUT_L"
-		(shape output)
+		(shape input)
 		(at 47.625 81.28 0)
 		(effects
