File: AudioBoard/AudioBoard/AudioBoard.kicad_pcb (KiCad board)
At the start: 4 copper layers, 250 x 160 mm, 310 parts, among them J1 IN, J2 XLR_L, J3 FX_RETURN, J4 FX_SEND, J5 INS_OUT, J6 XLR_R, J7_PWR_IN1 HC-DC-005-2.0T, J8 NMJ6HFD2, J9 NMJ6HFD2, SW2 SW_SPDT_321, SW3_pwr1 SS-12D28G7, U10 TL072, U11 TL072, U12 AMS1117-3.3, U13 AMS1117-3.3, U14 TL072, U15 NJM4556A, U16 TL072, U17 TL072, U18 NJM4556A, U19 TL072, U2 NE5532, U20 TL072, U21 TPS7A39, U22 URA2415S-6WR3, U24 TURB2405YMD-30WR3, U3 TPS26600PWP, U4 TL072, U5 TL072, U6 TL072, U7 TL072, U8 TL072, U9 TL072

Commit message: added bias voltage buffer, fixed fsw shift reg input filter
Parts:
- added C102: 100nF, Capacitor_SMD:C_0603_1608Metric, F.Cu at (81.2, 74.2)
- added C103: 100uF, Capacitor_SMD:CP_Elec_5x5.4, F.Cu at (128.8, 161.5)
- added C104: 100uF, Capacitor_SMD:CP_Elec_5x5.4, F.Cu at (128.8, 168.4)
- added C105: 100uF, Capacitor_SMD:CP_Elec_5x5.4, F.Cu at (128.8, 175.2)
- added C107: 100uF, Capacitor_SMD:CP_Elec_5x5.4, F.Cu at (128.8, 182.1)
- added C138: 100uF, Capacitor_SMD:CP_Elec_5x5.4, F.Cu at (128.8, 188.9)
- added C139: 100uF, Capacitor_SMD:CP_Elec_5x5.4, F.Cu at (128.8, 195.8)
- added C141: 4.7uF, Capacitor_SMD:C_1206_3216Metric, F.Cu at (59.0, 90.4)
- added C142: 100uF, Capacitor_SMD:CP_Elec_5x5.4, F.Cu at (55.8, 112.4)
- added C143: 100uF, Capacitor_SMD:CP_Elec_5x5.4, F.Cu at (55.8, 106.0)
- added C144: 100n, Capacitor_SMD:C_0402_1005Metric, F.Cu at (177.2, 183.4)
- added C145: 100n, Capacitor_SMD:C_0402_1005Metric, F.Cu at (177.2, 185.4)
- added C147: 100n, Capacitor_SMD:C_0402_1005Metric, F.Cu at (203.6, 187.1)
- added C148: 100n, Capacitor_SMD:C_0402_1005Metric, F.Cu at (197.6, 187.1)
- added C149: 100n, Capacitor_SMD:C_0402_1005Metric, F.Cu at (191.6, 180.7)
- added C160: 100n, Capacitor_SMD:C_0402_1005Metric, F.Cu at (203.6, 180.7)
- added C161: 100n, Capacitor_SMD:C_0402_1005Metric, F.Cu at (191.6, 187.1)
- added C162: 100n, Capacitor_SMD:C_0402_1005Metric, F.Cu at (197.6, 180.7)
- added C163: 100n, Capacitor_SMD:C_0402_1005Metric, F.Cu at (191.6, 193.6)
- added C164: 100n, Capacitor_SMD:C_0402_1005Metric, F.Cu at (197.6, 193.6)
- added C165: 100n, Capacitor_SMD:C_0402_1005Metric, F.Cu at (217.4, 191.5)
- added C166: 100n, Capacitor_SMD:C_0402_1005Metric, F.Cu at (211.4, 191.5)
- added C167: 100n, Capacitor_SMD:C_0402_1005Metric, F.Cu at (195.7, 201.4)
- added C168: 100n, Capacitor_SMD:C_0402_1005Metric, F.Cu at (211.4, 185.1)
- added C169: 100n, Capacitor_SMD:C_0402_1005Metric, F.Cu at (217.4, 185.1)
- added C170: 100n, Capacitor_SMD:C_0402_1005Metric, F.Cu at (195.7, 207.9)
- added C171: 100n, Capacitor_SMD:C_0402_1005Metric, F.Cu at (223.4, 185.1)
- added C172: 100n, Capacitor_SMD:C_0402_1005Metric, F.Cu at (223.4, 191.5)
- added C56: 1uF, Capacitor_SMD:C_0603_1608Metric, F.Cu at (60.0, 78.2)
- added J11: USB_C_Receptacle_USB2.0, Connector_USB:USB_C_Receptacle_XKB_U262-16XN-4BVC11, F.Cu at (81.5, 63.7)
- added J7: Conn_02x10_FSW, Connector_PinSocket_1.27mm:PinSocket_2x10_P1.27mm_Vertical, F.Cu at (200.4, 202.1)
- added R1: 39k, Resistor_SMD:R_0603_1608Metric, F.Cu at (135.3, 159.4)
- added R100: 1k, Resistor_SMD:R_0603_1608Metric, F.Cu at (204.2, 184.9)
- added R103: 1k, Resistor_SMD:R_0603_1608Metric, F.Cu at (198.2, 184.9)
- added R104: 1k, Resistor_SMD:R_0603_1608Metric, F.Cu at (192.2, 178.4)
- added R105: 1k, Resistor_SMD:R_0603_1608Metric, F.Cu at (204.2, 178.4)
- added R106: 1k, Resistor_SMD:R_0603_1608Metric, F.Cu at (192.2, 184.9)
- added R107: 1k, Resistor_SMD:R_0603_1608Metric, F.Cu at (198.2, 178.4)
- added R108: 1k, Resistor_SMD:R_0603_1608Metric, F.Cu at (192.2, 191.4)
- added R109: 1k, Resistor_SMD:R_0603_1608Metric, F.Cu at (198.2, 191.4)
- added R110: 1k, Resistor_SMD:R_0603_1608Metric, F.Cu at (218.0, 189.3)
- added R111: 1k, Resistor_SMD:R_0603_1608Metric, F.Cu at (212.0, 189.3)
- added R112: 1k, Resistor_SMD:R_0603_1608Metric, F.Cu at (196.2, 199.2)
- added R113: 1k, Resistor_SMD:R_0603_1608Metric, F.Cu at (212.0, 182.8)
- added R114: 1k, Resistor_SMD:R_0603_1608Metric, F.Cu at (218.0, 182.8)
- added R115: 1k, Resistor_SMD:R_0603_1608Metric, F.Cu at (196.2, 205.7)
- added R116: 1k, Resistor_SMD:R_0603_1608Metric, F.Cu at (224.0, 182.8)
- added R139: 1k, Resistor_SMD:R_0603_1608Metric, F.Cu at (224.0, 189.3)
- added R2: 51k, Resistor_SMD:R_0603_1608Metric, F.Cu at (135.3, 161.9)
- added R25: 10k, Resistor_SMD:R_0603_1608Metric, F.Cu at (135.3, 166.9)
- added R3: 100k, Resistor_SMD:R_0402_1005Metric, F.Cu at (134.7, 169.1)
- added R47: 5.6k, Resistor_SMD:R_0603_1608Metric, F.Cu at (56.8, 89.6)
- added R48: 30k, Resistor_SMD:R_0805_2012Metric, F.Cu at (54.8, 88.6)
- added R49: 100k, Resistor_SMD:R_0402_1005Metric, F.Cu at (61.4, 88.1)
- added R50: 20k, Resistor_SMD:R_0603_1608Metric, F.Cu at (62.0, 89.5)
- added R51: 0R, Resistor_SMD:R_0603_1608Metric_Pad0.98x0.95mm_HandSolder, F.Cu at (63.2, 79.6)
- added R52: 100k, Resistor_SMD:R_0402_1005Metric, F.Cu at (66.8, 76.4)
- added R53: 20k, Resistor_SMD:R_0603_1608Metric, F.Cu at (66.8, 79.0)
- added R54: 0R, Resistor_SMD:R_0603_1608Metric_Pad0.98x0.95mm_HandSolder, F.Cu at (62.8, 95.8)
- added R55: 0R, Resistor_SMD:R_0603_1608Metric_Pad0.98x0.95mm_HandSolder, F.Cu at (61.2, 95.8)
- added R7: 10k, Resistor_SMD:R_0603_1608Metric, F.Cu at (135.3, 164.4)
- added U23: USBLC6-2P6, Package_TO_SOT_SMD:SOT-666, F.Cu at (81.2, 70.9)
- added U26: 74HC165, Package_SO:SOIC-16_3.9x9.9mm_P1.27mm, F.Cu at (172.5, 193.3)
- added U27: 74HC165, Package_SO:SOIC-16_3.9x9.9mm_P1.27mm, F.Cu at (180.9, 193.3)
- R143, R144, R145, R146: value 100 -> 100R; footprint Resistor_SMD:R_0603_1608Metric -> Resistor_SMD:R_0402_1005Metric
- R27, R34, R35, R43: footprint Resistor_SMD:R_0402_1005Metric -> Resistor_SMD:R_0603_1608Metric_Pad0.98x0.95mm_HandSolder
- moved U3 128.2 mm to (59.4, 83.4), turned to -90 degrees
- moved C61 104.0 mm to (73.8, 91.9), turned to -90 degrees
- moved FB2 93.2 mm to (60.8, 102.6), turned to -90 degrees
- moved U12 64.1 mm to (62.2, 190.2)
- moved FB1 60.8 mm to (55.4, 187.6)
- moved C62 59.5 mm to (56.6, 191.8)
- moved C81 57.0 mm to (55.2, 189.8), turned to 180 degrees
- moved C85 56.4 mm to (57.0, 183.6), turned to -90 degrees
- moved U13 54.4 mm to (62.1, 181.8)
- moved C86 53.9 mm to (55.1, 182.2), turned to 90 degrees
- moved C100 52.9 mm to (55.0, 155.0), turned to 180 degrees
- moved C99 52.2 mm to (55.0, 153.8), turned to 180 degrees
- moved C82 50.7 mm to (71.4, 189.1), turned to -90 degrees
- moved FB3 48.0 mm to (54.6, 157.4), turned to -90 degrees
- moved U24 44.1 mm to (62.5, 128.5), turned to 0 degrees
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Connections:
- net /power/+5V renamed +5V
- R118 pad 1: /HeadphoneAmplifier1/OUT -> /Audio_IO_conn/HEADPHONE_L
- R120 pad 1: /HeadphoneAmplifier1/OUT -> /Audio_IO_conn/HEADPHONE_L
Routing:
- net GNDPWR: track 95.2 -> 15.9 mm, vias 0 -> 1
- net +5V: track 0.00 -> 46.7 mm
- net /power/AnalogPower/VIN: track 0.00 -> 29.1 mm
- net /power/input_pwr_protection/VIN: track 0.00 -> 19.8 mm
- net /power/input_pwr_protection/\SHDN: track 0.00 -> 16.1 mm, vias 0 -> 1
- net Net-(U24-+Vin): track 0.00 -> 10.3 mm
- net Net-(U12-VI): track 0.00 -> 6.55 mm
- net Net-(U3-~{FLT}): track 0.00 -> 5.37 mm
- net Net-(SW3_pwr1-B): track 0.00 -> 5.17 mm
- net /usb_interface/USB_Conn_D+: track 0.00 -> 5.14 mm
- net /usb_interface/USB_Conn_D-: track 0.00 -> 4.60 mm
- net GND: track 80.1 -> 84.5 mm, vias 82 -> 85
- net Net-(U3-IMON): track 0.00 -> 4.13 mm
- net Net-(U3-ILIM): track 0.00 -> 3.19 mm
- net Net-(U24-+Vout): track 0.00 -> 2.83 mm
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