File: AudioBoard/AudioBoard/input_pwr_protection.kicad_sch (KiCad schematic)
At the start: 10 parts, among them U3 TPS26600PWP

Commit message: assigned footprint to elements lcsc parts
Parts:
- C141: footprint (none) -> Capacitor_SMD:C_1206_3216Metric; JLCPCB (none) -> C29823; LCSC Part (none) -> C29823
- C56: footprint (none) -> Capacitor_SMD:C_0603_1608Metric; JLCPCB (none) -> C15849; LCSC Part (none) -> C15849
- C61: JLCPCB (none) -> C105334; LCSC Part (none) -> C105334
- R47: footprint (none) -> Resistor_SMD:R_0603_1608Metric; JLCPCB (none) -> C23189; LCSC Part (none) -> C23189
- R48: footprint (none) -> Resistor_SMD:R_0805_2012Metric; JLCPCB (none) -> C17621; LCSC Part (none) -> C17621
- R49: footprint (none) -> Resistor_SMD:R_0402_1005Metric; JLCPCB (none) -> C25741; LCSC Part (none) -> C25741
- R50: footprint (none) -> Resistor_SMD:R_0603_1608Metric; JLCPCB (none) -> C4184; LCSC Part (none) -> C4184
- R51, R55: footprint (none) -> Resistor_SMD:R_0603_1608Metric_Pad0.98x0.95mm_HandSolder; JLCPCB (none) -> C21189; LCSC Part (none) -> C21189
- U3: JLCPCB (none) -> C544399; LCSC Part (none) -> C544399

Commit message: added bias voltage buffer, fixed fsw shift reg input filter
Parts:
- R51: now left out of the parts list
Changed lines of the file:
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@@
 		(lib_id "Device:C_Polarized")
 		(at 94.615 76.2 0)
+		(mirror y)
 		(unit 1)
 		(body_style 1)
@@
 		(in_pos_files yes)
 		(dnp no)
-		(fields_autoplaced yes)
 		(property "Reference" "C61"
-			(at 98.425 74.0409 0)
+			(at 90.805 74.0409 0)
 			(show_name no)
 			(do_not_autoplace no)
@@
 		)
 		(property "Value" "2200uF"
-			(at 98.425 76.5809 0)
+			(at 90.805 76.5809 0)
 			(show_name no)
 			(do_not_autoplace no)
@@
 		)
 		(property "Footprint" "Capacitor_THT:C_Radial_D16.0mm_H25.0mm_P7.50mm"
-			(at 95.5802 80.01 0)
+			(at 93.6498 80.01 0)
 			(hide yes)
 			(show_name no)
@@
 		(body_style 1)
 		(exclude_from_sim no)
-		(in_bom yes)
+		(in_bom no)
 		(on_board yes)
 		(in_pos_files yes)
