File: AudioBoard/AudioBoard/Instrument_Input.kicad_sch (KiCad schematic)
At the start: 25 parts, among them U6 TL072

Commit message: modified clamping diodes on inputs, added exp pedal input filter, added ideas to instrument input filter redesign
Parts:
- removed C15, C18: 100n, Capacitor_SMD:C_0402_1005Metric, symbol Device:C_Small
- removed D5, D6, D7, D8: 1N4148W, Diode_SMD:D_SOD-123, symbol Diode:1N4148W
- added D20, D23: BAT54S, Package_TO_SOT_SMD:SOT-23, symbol Diode:BAT54S
Connections:
- net AVDD: now also D20.2 (K), D23.2 (K)
- net GND: now also D20.1 (A), D23.1 (A)
- net OUT_N: now also D23.3 (COM)
- net OUT_P: now also D20.3 (COM)
